Commit message: mi laser scan

File: summit_description/urdf/base/summit_base.gazebo.xacro (robot description, xacro)
@@ -14,10 +14,10 @@
 	    </plugin>
 	  </gazebo>
-	<!-- hokuyo -->
-  <gazebo reference="hokuyo">
-    <sensor type="gpu_ray" name="head_hokuyo_sensor">
+  <!-- Hukuyo Laser Plugin -->
+  <gazebo reference="laser_link">
+    <sensor type="ray" name="head_hokuyo_sensor">
       <pose>0 0 0 0 0 0</pose>
       <visualize>false</visualize>
-      <update_rate>40</update_rate>
+      <update_rate>20</update_rate>
       <ray>
         <scan>
@@ -25,6 +25,8 @@
             <samples>720</samples>
             <resolution>1</resolution>
-            <min_angle>-1.570796</min_angle>
-            <max_angle>1.570796</max_angle>
+            <!--<min_angle>-1.570796</min_angle>
+            <max_angle>1.570796</max_angle>-->
+            <min_angle>-3.14159</min_angle>
+            <max_angle>3.14159</max_angle>
           </horizontal>
         </scan>
@@ -32,17 +34,13 @@
           <min>0.10</min>
           <max>20.0</max>
-          <resolution>0.05</resolution>
+          <resolution>0.01</resolution>
         </range>
         <noise>
           <type>gaussian</type>
-          <!-- Noise parameters based on published spec for Hokuyo laser
-               achieving "+-30mm" accuracy at range < 10m.  A mean of 0.0m and
-               stddev of 0.01m will put 99.7% of samples within 0.03m of the true
-               reading. -->
           <mean>0.0</mean>
           <stddev>0.01</stddev>
         </noise>
       </ray>
-      <plugin name="gazebo_ros_head_hokuyo_controller" filename="libgazebo_ros_gpu_laser.so">
+      <plugin name="gazebo_ros_head_hokuyo_controller" filename="libgazebo_ros_laser.so">
         <topicName>/scan</topicName>
         <frameName>/laser_link</frameName>

File: summit_description/urdf/base/summit_base.urdf.xacro (robot description, xacro)
@@ -43,10 +43,4 @@
     </collision>
   </link>
-  <joint name="hokuyo_joint" type="fixed">
-    <axis xyz="0 1 0" />
-    <origin xyz="0 0 0.435" rpy="0 0 0"/>
-    <parent link="base_link"/>
-    <child link="laser_link"/>
-  </joint>
   <!-- Hokuyo Laser -->
   <link name="laser_link">
@@ -60,5 +54,6 @@
       <origin xyz="0 0 0" rpy="0 0 0"/>
       <geometry>
-        <mesh filename="package://summit_description/meshes/hokuyo/hokuyo.dae"/>
+        <!-- <mesh filename="package://summit_description/meshes/hokuyo/hokuyo.dae"/> -->
+    <box size="0.1 0.1 0.1"/>
       </geometry>
     </visual>
@@ -69,4 +64,10 @@
     </inertial>
   </link>
+  <joint name="hokuyo_joint" type="fixed">
+    <axis xyz="0 1 0" />
+    <origin xyz="0 0 0.435" rpy="0 0 0"/>
+    <parent link="base_link"/>
+    <child link="laser_link"/>
+  </joint>
   </xacro:macro>
 </robot>
