Commit message: two_part_world

File: src/simulation_environment/models/diff_drive/parameter.xacro (robot description, xacro)
@@ -9,5 +9,5 @@
   <xacro:property name="y_chassis" value="0.3" />
   <xacro:property name="z_chassis" value="0.15" />
-  <xacro:property name="m_chassis" value="10.0" />
+  <xacro:property name="m_chassis" value="20.0" />
   <!-- Parameter for the wheels, radius [m], height [m], mass [kg], torque [Nm], wheelbase [m] -->
   <xacro:property name="r_wheel" value="${properties['wheel_radius']}"/>

Commit message: launch

File: src/simulation_environment/models/diff_drive/parameter.xacro (robot description, xacro)
@@ -9,5 +9,5 @@
   <xacro:property name="y_chassis" value="0.3" />
   <xacro:property name="z_chassis" value="0.15" />
-  <xacro:property name="m_chassis" value="20.0" />
+  <xacro:property name="m_chassis" value="10.0" />
   <!-- Parameter for the wheels, radius [m], height [m], mass [kg], torque [Nm], wheelbase [m] -->
   <xacro:property name="r_wheel" value="${properties['wheel_radius']}"/>
